File: PCB/cherry-hotswap/corne73.kicad_pcb (KiCad board)
At the start: 2 copper layers, 277.2 x 107.5 mm, 101 parts, among them J1 TYPE-C-31-M-13C, J3 Conn_01x04, J4 Conn_01x03, J5 TC2030_SWD, J6 Battery, Q1 AO3401A, SW1 SW_Push, SW10 SW_Push, SW11 SW_Push, SW12 SW_Push, SW13 SW_Push, SW14 SW_Push, SW15 SW_Push, SW16 SW_Push, SW17 SW_Push, SW18 SW_Push, SW19 SW_Push, SW2 SW_Push, SW20 SW_Push, SW21 SW_Push, SW22 SW_SPDT, SW23 SW_Push, SW3 SW_Push, SW4 SW_Push, SW5 SW_Push, SW6 SW_Push, SW7 SW_Push, SW8 SW_Push, SW9 SW_Push, U1 nRF52840_E73-2G4M08S1C, U2 TP4056, U3 USBLC6-2SC6, Y1 32.768 KHz

Commit message: Catching up
Parts:
- removed J3: Conn_01x04, kbd_local:OLED
- removed J4: Conn_01x03, Connector_PinHeader_2.54mm:PinHeader_1x03_P2.54mm_Vertical
- removed R3: 806, Resistor_SMD:R_0603_1608Metric
- removed R4: 2M, Resistor_SMD:R_0603_1608Metric
- removed ZD1: RB521S30T1G, Diode_SMD:D_SOD-523
- added D10: 1N4148, qw-footprints:CUSTOM D_SOD-123, B.Cu at (-93.6, 8.88)
- added D11: 1N4148, qw-footprints:CUSTOM D_SOD-123, B.Cu at (-74.6, 6.50)
- added D12: 1N4148, qw-footprints:CUSTOM D_SOD-123, B.Cu at (-55.5, 8.88)
- added D13: 1N4148, qw-footprints:CUSTOM D_SOD-123, B.Cu at (-40.9, 11.0)
- added D14: 1N4148, qw-footprints:CUSTOM D_SOD-123, B.Cu at (-131.7, 32.7)
- added D15: 1N4148, qw-footprints:CUSTOM D_SOD-123, B.Cu at (-112.7, 32.7)
- added D16: 1N4148, qw-footprints:CUSTOM D_SOD-123, B.Cu at (-93.6, 27.9)
- added D17: 1N4148, qw-footprints:CUSTOM D_SOD-123, B.Cu at (-78.8, 17.3)
- added D18: 1N4148, qw-footprints:CUSTOM D_SOD-123, B.Cu at (-59.7, 19.7)
- added D19: 1N4148, qw-footprints:CUSTOM D_SOD-123, B.Cu at (-36.5, 30.3)
- added D2: 1N4148, qw-footprints:CUSTOM D_SOD-123, B.Cu at (-131.7, -5.40)
- added D20: 1N4148, qw-footprints:CUSTOM D_SOD-123, B.Cu at (-54.5, 54.5)
- added D21: 1N4148, qw-footprints:CUSTOM D_SOD-123, B.Cu at (-35.3, 57.9)
- added D22: 1N4148, qw-footprints:CUSTOM D_SOD-123, B.Cu at (-23.8, 62.2)
- added D23: 1N4148, qw-footprints:CUSTOM D_SOD-123, B.Cu at (-17.5, 3.32)
- added D24: 1N4148, qw-footprints:CUSTOM D_SOD-123, B.Cu at (-17.6, 22.2)
- added D3: 1N4148, qw-footprints:CUSTOM D_SOD-123, B.Cu at (-112.7, -5.40)
- added D4: 1N4148, qw-footprints:CUSTOM D_SOD-123, B.Cu at (-93.6, -10.2)
- added D5: 1N4148, qw-footprints:CUSTOM D_SOD-123, B.Cu at (-74.6, -12.5)
- added D6: 1N4148, qw-footprints:CUSTOM D_SOD-123, B.Cu at (-55.5, -10.2)
- added D7: 1N4148, qw-footprints:CUSTOM D_SOD-123, B.Cu at (-36.5, -7.79)
- added D8: 1N4148, qw-footprints:CUSTOM D_SOD-123, B.Cu at (-131.7, 13.6)
- added D9: 1N4148, qw-footprints:CUSTOM D_SOD-123, B.Cu at (-112.7, 13.6)
- added F1: Fuse_Small, Fuse:Fuse_1206_3216Metric, B.Cu at (-23.2, -10.6)
- added J2: nice!view, Connector_PinHeader_2.54mm:PinHeader_1x05_P2.54mm_Vertical, F.Cu at (-9.21, 28.8)
- SW1, rSW1: footprint kbd:keyswitch_cherrymx_hotswap_1.5u -> PCM_marbastlib-mx:SW_MX_HS_CPG151101S11_1.5u
- SW10, SW11, SW12, SW13, SW14, SW15, SW16, SW17, SW18, SW19, SW2, SW20, SW21, SW3, SW4, SW5, SW6, SW7, SW8, SW9, rSW10, rSW11, rSW12, rSW13, rSW14, rSW15, rSW16, rSW17, rSW18, rSW19, rSW2, rSW20, rSW21, rSW3, rSW4, rSW5, rSW6, rSW7, rSW8, rSW9: footprint kbd:keyswitch_cherrymx_hotswap_1u -> PCM_marbastlib-mx:SW_MX_HS_CPG151101S11_1u
- moved H3 197.0 mm to (-7.69, 6.95)
- moved R5 189.9 mm to (-30.2, -49.1)
- moved LED1 180.8 mm to (-30.6, -44.2)
- moved R6 179.4 mm to (-13.5, 37.9)
- moved H7 177.8 mm to (-27.8, 42.9)
- moved D1 176.1 mm to (-14.2, 35.4), turned to -90 degrees
- moved Q1 165.5 mm to (-11.2, 35.4), turned to 0 degrees
- moved C8 164.6 mm to (-26.7, 13.8), turned to 90 degrees
- moved R7 160.4 mm to (-36.3, 18.0), turned to -90 degrees
- moved C7 156.2 mm to (-36.3, 13.9), turned to 90 degrees
- moved C6 153.0 mm to (-37.9, 13.9), turned to 90 degrees
- moved J6 150.8 mm to (-23.7, 28.3)
- moved Y1 136.1 mm to (-55.7, 31.6), turned to 90 degrees
- moved L1 133.3 mm to (-55.6, 39.9), turned to 0 degrees
- moved C5 133.0 mm to (-55.6, 38.5), turned to 0 degrees
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Connections:
- EXSW1 pad S1: GND -> Net-(D23-A)
- EXSW1 pad S2: /left/KEYEX1 -> unconnected-(EXSW1-PadS2)
- EXSW2 pad S1: GND -> Net-(D24-A)
- EXSW2 pad S2: /left/KEYEX2 -> unconnected-(EXSW2-PadS2)
- Q1 pad 3: BATTTON -> Net-(Q1-D)
- SW1 pad 1: /left/KEY1 -> Net-(D22-A)
- SW1 pad 2: GND -> Net-(SW1-Pad2)
- SW10 pad 1: /left/KEY10 -> Net-(D17-A)
- SW10 pad 2: GND -> Net-(SW10-Pad2)
- SW11 pad 1: /left/KEY11 -> Net-(D11-A)
- SW11 pad 2: GND -> Net-(SW10-Pad2)
- SW12 pad 1: /left/KEY12 -> Net-(D5-A)
- SW12 pad 2: GND -> Net-(SW10-Pad2)
- SW13 pad 1: /left/KEY13 -> Net-(D4-A)
- SW13 pad 2: GND -> Net-(SW13-Pad2)
- SW14 pad 1: /left/KEY14 -> Net-(D10-A)
- SW14 pad 2: GND -> Net-(SW13-Pad2)
- SW15 pad 1: /left/KEY15 -> Net-(D16-A)
- SW15 pad 2: GND -> Net-(SW13-Pad2)
- SW16 pad 1: /left/KEY16 -> Net-(D15-A)
- SW16 pad 2: GND -> Net-(SW16-Pad2)
- SW17 pad 1: /left/KEY17 -> Net-(D9-A)
- SW17 pad 2: GND -> Net-(SW16-Pad2)
- SW18 pad 1: /left/KEY18 -> Net-(D3-A)
- SW18 pad 2: GND -> Net-(SW16-Pad2)
- SW19 pad 1: /left/KEY19 -> Net-(D2-A)
- SW19 pad 2: GND -> Net-(SW19-Pad2)
- SW2 pad 1: /left/KEY2 -> Net-(D19-A)
- SW2 pad 2: GND -> Net-(SW1-Pad2)
- SW20 pad 1: /left/KEY20 -> Net-(D8-A)
- SW20 pad 2: GND -> Net-(SW19-Pad2)
- SW21 pad 1: /left/KEY21 -> Net-(D14-A)
- SW21 pad 2: GND -> Net-(SW19-Pad2)
- SW22 pad 1: unconnected-(SW22-A-Pad1) -> +BATT
- SW22 pad 2: unconnected-(SW22-B-Pad2) -> Net-(Q1-D)
- SW23 pad 1: unconnected-(SW23-Pad1) -> RESET
- SW23 pad 2: unconnected-(SW23-Pad2) -> GND
- SW3 pad 1: /left/KEY3 -> Net-(D13-A)
- SW3 pad 2: GND -> Net-(SW1-Pad2)
- SW4 pad 1: /left/KEY4 -> Net-(D7-A)
- SW4 pad 2: GND -> Net-(SW1-Pad2)
- SW5 pad 1: /left/KEY5 -> Net-(D6-A)
- SW5 pad 2: GND -> Net-(SW5-Pad2)
- SW6 pad 1: /left/KEY6 -> Net-(D12-A)
- SW6 pad 2: GND -> Net-(SW5-Pad2)
- SW7 pad 1: /left/KEY7 -> Net-(D18-A)
- SW7 pad 2: GND -> Net-(SW5-Pad2)
- SW8 pad 1: /left/KEY8 -> Net-(D21-A)
- SW8 pad 2: GND -> Net-(SW5-Pad2)
- SW9 pad 1: /left/KEY9 -> Net-(D20-A)
- SW9 pad 2: GND -> Net-(SW10-Pad2)
- U1 pad 1: 1.11 -> unconnected-(U1-P1.11-Pad1)
- U1 pad 10: 0.30 -> unconnected-(U1-P0.30/AIN6-Pad10)
- U1 pad 12: 0.26 -> unconnected-(U1-P0.26-Pad12)
- U1 pad 14: 0.06 -> CS
- U1 pad 15: VSENSE -> unconnected-(U1-P0.05/AIN3-Pad15)
- U1 pad 16: 0.08 -> unconnected-(U1-P0.08-Pad16)
- U1 pad 17: 1.09 -> unconnected-(U1-P1.09-Pad17)
- U1 pad 18: 0.04 -> unconnected-(U1-P0.04/AIN2-Pad18)
- U1 pad 2: 1.10 -> unconnected-(U1-P1.10-Pad2)
- U1 pad 20: 0.12 -> unconnected-(U1-P0.12-Pad20)
- U1 pad 22: 0.07 -> unconnected-(U1-P0.07-Pad22)
- U1 pad 28: 0.15 -> unconnected-(U1-P0.15-Pad28)
- U1 pad 3: 0.03 -> unconnected-(U1-P0.03/AIN1-Pad3)
- U1 pad 30: 0.17 -> MOSI
- U1 pad 32: 0.20 -> SCK
- U1 pad 33: 0.13 -> unconnected-(U1-P0.13-Pad33)
- U1 pad 34: 0.22 -> unconnected-(U1-P0.22-Pad34)
- U1 pad 35: 0.24 -> unconnected-(U1-P0.24-Pad35)
- U1 pad 36: 1.00 -> unconnected-(U1-P1.00-Pad36)
- U1 pad 38: 1.02 -> unconnected-(U1-P1.02-Pad38)
- U1 pad 4: 0.28 -> unconnected-(U1-P0.28/AIN4-Pad4)
- U1 pad 40: 1.04 -> unconnected-(U1-P1.04-Pad40)
- U1 pad 41: 0.09 -> unconnected-(U1-P0.09/NFC1-Pad41)
- U1 pad 42: 1.06 -> unconnected-(U1-P1.06-Pad42)
- U1 pad 43: 0.10 -> unconnected-(U1-P0.10/NFC2-Pad43)
- U1 pad 6: 1.13 -> unconnected-(U1-P1.13-Pad6)
- U1 pad 7: 0.02 -> unconnected-(U1-P0.02/AIN0-Pad7)
- U1 pad 8: 0.29 -> unconnected-(U1-P0.29/AIN5-Pad8)
- U1 pad 9: 0.31 -> unconnected-(U1-P0.31/AIN7-Pad9)
- U3 pad 1: DBUS- -> D+
- U3 pad 4: D+ -> DBUS-
Routing:
- net +5V: track 0.00 -> 150.1 mm, vias 0 -> 5
- net Net-(D10-K): track 0.00 -> 125.5 mm, vias 0 -> 2
- net Net-(D2-K): track 0.00 -> 102.8 mm
- net Net-(D14-K): track 0.00 -> 91.9 mm
- net D+: track 0.00 -> 86.7 mm
- net D-: track 0.00 -> 85.4 mm
- net +VSW: track 0.00 -> 53.9 mm, vias 0 -> 2
- net Net-(SW16-Pad2): track 0.00 -> 38.6 mm
- net Net-(SW13-Pad2): track 0.00 -> 38.6 mm
- net Net-(SW19-Pad2): track 0.00 -> 38.6 mm
- net Net-(SW5-Pad2): track 0.00 -> 38.6 mm
- net Net-(SW10-Pad2): track 0.00 -> 38.6 mm
- net +BATT: track 0.00 -> 38.5 mm
- net DBUS+: track 0.00 -> 26.4 mm, vias 0 -> 2
- net DBUS-: track 0.00 -> 25.4 mm, vias 0 -> 2
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- added copper zone on B.Cu, net GND
- added copper zone on F.Cu, net GND
Other:
- rule pad_to_mask_clearance: 0.2 -> 0.05
- board text added: "Corne73 by quark https://quark.works/ 19.99"
- board text added: "ON OFF"

Commit message: Changed footprints, made decisions
Parts:
- D1: footprint Diode_SMD:D_SOD-323 -> Corne73:D_SOD-123
- D10, D11, D12, D13, D14, D15, D16, D17, D18, D19, D2, D20, D21, D22, D23, D24, D3, D4, D5, D6, D7, D8, D9: footprint qw-footprints:CUSTOM D_SOD-123 -> Corne73:D_SOD-123
- SW1: footprint PCM_marbastlib-mx:SW_MX_HS_CPG151101S11_1.5u -> Corne73:SwitchCombo; moved to F.Cu
- SW10, SW11, SW12, SW13, SW14, SW15, SW16, SW17, SW18, SW19, SW2, SW20, SW21, SW3, SW4, SW5, SW6, SW7, SW8, SW9: footprint PCM_marbastlib-mx:SW_MX_HS_CPG151101S11_1u -> Corne73:SwitchCombo; moved to F.Cu
- rSW1: footprint PCM_marbastlib-mx:SW_MX_HS_CPG151101S11_1.5u -> Corne73:SwitchCombo
- rSW10, rSW11, rSW12, rSW13, rSW14, rSW15, rSW16, rSW17, rSW18, rSW19, rSW2, rSW20, rSW21, rSW3, rSW4, rSW5, rSW6, rSW7, rSW8, rSW9: footprint PCM_marbastlib-mx:SW_MX_HS_CPG151101S11_1u -> Corne73:SwitchCombo
- moved H7 145.7 mm to (-173.5, 39.3)
- moved C8 20.8 mm to (-17.2, 32.4), turned to 0 degrees
- moved C7 19.6 mm to (-27.7, 31.5)
- moved C6 19.6 mm to (-29.3, 31.5)
- moved R7 19.6 mm to (-27.7, 35.6)
- moved U2 19.6 mm to (-23.0, 34.3)
- moved J6 1.63 mm to (-23.7, 26.7), turned to 0 degrees
- moved R6 0.57 mm to (-13.5, 38.5)
- moved D13 0.18 mm to (-41.1, 11.0)
- moved D19 0.18 mm to (-36.7, 30.3)
- moved D7 0.18 mm to (-36.7, -7.79)
- moved D10 0.17 mm to (-93.8, 8.88)
- moved D11 0.17 mm to (-74.8, 6.50)
- moved D12 0.17 mm to (-55.7, 8.88)
- moved D15 0.17 mm to (-112.9, 32.7)
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Routing:
- net +BATT: track 38.5 -> 21.8 mm
- net +5V: track 150.1 -> 134.4 mm
- net Net-(D3-A): track 2.90 -> 7.98 mm
- net Net-(D2-A): track 2.90 -> 7.91 mm
- net GND: track 22.3 -> 25.3 mm, vias 8 -> 9
- net Net-(SW16-Pad2): track 38.6 -> 41.4 mm
- net Net-(SW19-Pad2): track 38.6 -> 41.3 mm

Commit message: More changes
Parts:
- removed rU3: TPD4E05U06DQAR, Package_SON:USON-10_2.5x1.0mm_P0.5mm
- EXSW1, EXSW2: footprint kbd_local:keyswitch_cherrymx_hotswap_1u_rotary_encoder_ec12 -> Corne73:SwitchCombo+Encoder; moved to F.Cu
- rSW10, rSW11, rSW12, rSW13, rSW14, rSW15, rSW16, rSW17, rSW18, rSW19, rSW2, rSW20, rSW21, rSW3, rSW4, rSW5, rSW6, rSW7: moved to F.Cu
- moved R5 91.7 mm to (-7.77, 39.8)
- moved LED1 88.8 mm to (-5.27, 40.8), turned to -90 degrees
- moved SW23 34.6 mm to (-51.6, 50.4), turned to -90 degrees
- moved D21 9.65 mm to (-44.5, 54.8)
- moved D13 4.42 mm to (-36.7, 11.3)
- moved D20 2.93 mm to (-57.1, 55.9), turned to 180 degrees
- moved D22 2.55 mm to (-23.5, 59.7)
- moved D23 1.58 mm to (-17.6, 1.74)
- moved D24 1.44 mm to (-17.6, 20.8)
- turned EXSW1 to 0 degrees
- turned EXSW2 to 0 degrees
- turned rSW10 to 0 degrees
- turned rSW11 to 0 degrees
- turned rSW12 to 0 degrees
- turned rSW13 to 0 degrees
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Connections:
- D24 pad 1: Net-(D20-K) -> Net-(D14-K)
- EXSW1 pad A: /left/RE0A -> CS
- EXSW1 pad B: /left/REB -> /left/RE0B
- EXSW1 pad S2: unconnected-(EXSW1-PadS2) -> Net-(EXSW1-PadS2)
- EXSW2 pad A: /left/RE1A -> SCK
- EXSW2 pad B: /left/REB -> MOSI
- EXSW2 pad S2: unconnected-(EXSW2-PadS2) -> Net-(EXSW1-PadS2)
- J5 pad 3: RESET -> unconnected-(J5-~{RST}-Pad3)
Routing:
- net Net-(EXSW1-PadS2): track 0.00 -> 86.4 mm, vias 0 -> 2
- net Net-(SW1-Pad2): track 0.00 -> 83.6 mm
- net CS: track 0.00 -> 67.5 mm, vias 0 -> 2
- net Net-(D14-K): track 91.9 -> 152.6 mm, vias 0 -> 2
- net Net-(SW5-Pad2): track 38.6 -> 87.0 mm
- net SCK: track 0.00 -> 46.5 mm, vias 0 -> 2
- net MOSI: track 0.00 -> 40.8 mm, vias 0 -> 2
- net /left/RE0B: track 0.00 -> 34.5 mm, vias 0 -> 2
- net VDD: track 11.0 -> 43.9 mm, vias 0 -> 2
- net Net-(D20-K): track 0.00 -> 32.6 mm
- net RESET: track 0.00 -> 17.3 mm, vias 0 -> 2
- net unconnected-(U1-P1.09-Pad17): track 0.00 -> 15.9 mm
- net Net-(U2-CHRG): track 0.00 -> 15.7 mm, vias 0 -> 2
- net unconnected-(U1-P0.05/AIN3-Pad15): track 0.00 -> 14.7 mm
- net Net-(D21-A): track 0.00 -> 11.8 mm
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
Commit message: Left hand routed
Parts:
- moved J5 1.94 mm to (-71.3, 48.2), turned to -90 degrees
- moved C5 0.10 mm to (-55.5, 38.4)
- moved C4 0.10 mm to (-55.5, 36.0)
- moved L1 0.10 mm to (-55.5, 39.9)
Connections:
- D10 pad 1: Net-(D10-K) -> ROW1
- D11 pad 1: Net-(D10-K) -> ROW1
- D12 pad 1: Net-(D10-K) -> ROW1
- D13 pad 1: Net-(D10-K) -> ROW1
- D14 pad 1: Net-(D14-K) -> ROW2
- D15 pad 1: Net-(D14-K) -> ROW2
- D16 pad 1: Net-(D14-K) -> ROW2
- D17 pad 1: Net-(D14-K) -> ROW2
- D18 pad 1: Net-(D14-K) -> ROW2
- D19 pad 1: Net-(D14-K) -> ROW2
- D2 pad 1: Net-(D2-K) -> ROW0
- D20 pad 1: Net-(D20-K) -> ROW3
- D21 pad 1: Net-(D20-K) -> ROW3
- D22 pad 1: Net-(D20-K) -> ROW3
- D23 pad 1: Net-(D10-K) -> ROW1
- D24 pad 1: Net-(D14-K) -> ROW2
- D3 pad 1: Net-(D2-K) -> ROW0
- D4 pad 1: Net-(D2-K) -> ROW0
- D5 pad 1: Net-(D2-K) -> ROW0
- D6 pad 1: Net-(D2-K) -> ROW0
- D7 pad 1: Net-(D2-K) -> ROW0
- D8 pad 1: Net-(D10-K) -> ROW1
- D9 pad 1: Net-(D10-K) -> ROW1
- EXSW1 pad S2: Net-(EXSW1-PadS2) -> COL6
- EXSW2 pad S2: Net-(EXSW1-PadS2) -> COL6
- SW1 pad 2: Net-(SW1-Pad2) -> COL5
- SW10 pad 2: Net-(SW10-Pad2) -> COL3
- SW11 pad 2: Net-(SW10-Pad2) -> COL3
- SW12 pad 2: Net-(SW10-Pad2) -> COL3
- SW13 pad 2: Net-(SW13-Pad2) -> COL2
- SW14 pad 2: Net-(SW13-Pad2) -> COL2
- SW15 pad 2: Net-(SW13-Pad2) -> COL2
- SW16 pad 2: Net-(SW16-Pad2) -> COL1
- SW17 pad 2: Net-(SW16-Pad2) -> COL1
- SW18 pad 2: Net-(SW16-Pad2) -> COL1
- SW19 pad 2: Net-(SW19-Pad2) -> COL0
- SW2 pad 2: Net-(SW1-Pad2) -> COL5
- SW20 pad 2: Net-(SW19-Pad2) -> COL0
- SW21 pad 2: Net-(SW19-Pad2) -> COL0
- SW3 pad 2: Net-(SW1-Pad2) -> COL5
- SW4 pad 2: Net-(SW1-Pad2) -> COL5
- SW5 pad 2: Net-(SW5-Pad2) -> COL4
- SW6 pad 2: Net-(SW5-Pad2) -> COL4
- SW7 pad 2: Net-(SW5-Pad2) -> COL4
- SW8 pad 2: Net-(SW5-Pad2) -> COL4
- SW9 pad 2: Net-(SW10-Pad2) -> COL3
- U1 pad 1: unconnected-(U1-P1.11-Pad1) -> COL3
- U1 pad 10: unconnected-(U1-P0.30/AIN6-Pad10) -> /left/RE0B
- U1 pad 12: unconnected-(U1-P0.26-Pad12) -> CS
- U1 pad 14: CS -> unconnected-(U1-P0.06-Pad14)
- U1 pad 15: unconnected-(U1-P0.05/AIN3-Pad15) -> SCK
- U1 pad 17: unconnected-(U1-P1.09-Pad17) -> MOSI
- U1 pad 2: unconnected-(U1-P1.10-Pad2) -> ROW2
- U1 pad 3: unconnected-(U1-P0.03/AIN1-Pad3) -> COL2
- U1 pad 30: MOSI -> unconnected-(U1-P0.17-Pad30)
- U1 pad 32: SCK -> unconnected-(U1-P0.20-Pad32)
- U1 pad 33: unconnected-(U1-P0.13-Pad33) -> ROW3
- U1 pad 35: unconnected-(U1-P0.24-Pad35) -> COL4
- U1 pad 4: unconnected-(U1-P0.28/AIN4-Pad4) -> COL1
- U1 pad 41: unconnected-(U1-P0.09/NFC1-Pad41) -> COL5
- U1 pad 6: unconnected-(U1-P1.13-Pad6) -> COL0
- U1 pad 7: unconnected-(U1-P0.02/AIN0-Pad7) -> ROW1
- U1 pad 8: unconnected-(U1-P0.29/AIN5-Pad8) -> ROW0
- U1 pad 9: unconnected-(U1-P0.31/AIN7-Pad9) -> COL6
Routing:
- net ROW2: track 0.00 -> 171.5 mm, vias 0 -> 4
- net Net-(D14-K): track 152.6 -> 0.00 mm, vias 2 -> 0
- net ROW1: track 0.00 -> 148.7 mm, vias 0 -> 2
- net ROW0: track 0.00 -> 148.0 mm, vias 0 -> 2
- net COL4: track 0.00 -> 147.4 mm, vias 0 -> 1
- net COL5: track 0.00 -> 147.4 mm, vias 0 -> 1
- net COL0: track 0.00 -> 133.0 mm
- net Net-(D10-K): track 128.8 -> 0.00 mm, vias 2 -> 0
- net COL1: track 0.00 -> 120.0 mm
- net COL6: track 0.00 -> 115.6 mm, vias 0 -> 2
- net COL3: track 0.00 -> 112.7 mm
- net Net-(D2-K): track 104.6 -> 0.00 mm
- net COL2: track 0.00 -> 96.6 mm
- net Net-(SW5-Pad2): track 87.0 -> 0.00 mm
- net Net-(EXSW1-PadS2): track 86.4 -> 0.00 mm, vias 2 -> 0
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
Commit message: Started work on right side
Parts:
- removed rJ2: TRS, kbd_local:PJ-398A-5A_PJ-399B-6A
- removed rJ3: Conn_01x04, kbd_local:OLED
- removed rJ4: Conn_01x03, Connector_PinHeader_2.54mm:PinHeader_1x03_P2.54mm_Vertical
- removed rZD1: RB521S30T1G, Diode_SMD:D_SOD-523
- added C10: 10uF, Capacitor_Tantalum_SMD:CP_EIA-2012-12_Kemet-R, B.Cu at (183.3, 87.6)
- added C11: 4.7u, Capacitor_SMD:C_0603_1608Metric, B.Cu at (181.7, 87.5)
- added C12: 10uF, Capacitor_Tantalum_SMD:CP_EIA-2012-12_Kemet-R, B.Cu at (180.8, 81.4)
- added C13: 12p, Capacitor_SMD:C_0603_1608Metric, B.Cu at (217.3, 79.3)
- added C14: 4.7u, Capacitor_SMD:C_0603_1608Metric, B.Cu at (233.8, 73.2)
- added C15: 4.7u, Capacitor_SMD:C_0603_1608Metric, B.Cu at (224.7, 75.4)
- added C16: 12p, Capacitor_SMD:C_0603_1608Metric, B.Cu at (218.3, 78.2)
- added C9: 1u, Capacitor_SMD:C_0603_1608Metric, B.Cu at (222.6, 77.5)
- added D25: Schottky, Corne73:D_SOD-123, B.Cu at (169.1, 85.6)
- added D26: 1N4148, Corne73:D_SOD-123, B.Cu at (283.2, 42.0)
- added D27: 1N4148, Corne73:D_SOD-123, B.Cu at (264.2, 42.0)
- added D28: 1N4148, Corne73:D_SOD-123, B.Cu at (245.1, 37.3)
- added D29: 1N4148, Corne73:D_SOD-123, B.Cu at (226.1, 34.9)
- added D30: 1N4148, Corne73:D_SOD-123, B.Cu at (207.0, 37.3)
- added D31: 1N4148, Corne73:D_SOD-123, B.Cu at (188.0, 39.7)
- added D32: 1N4148, Corne73:D_SOD-123, B.Cu at (283.2, 61.1)
- added D33: 1N4148, Corne73:D_SOD-123, B.Cu at (264.2, 61.1)
- added D34: 1N4148, Corne73:D_SOD-123, B.Cu at (245.1, 56.3)
- added D35: 1N4148, Corne73:D_SOD-123, B.Cu at (226.1, 54.0)
- added D36: 1N4148, Corne73:D_SOD-123, B.Cu at (207.0, 56.3)
- added D37: 1N4148, Corne73:D_SOD-123, B.Cu at (188.0, 58.7)
- added D38: 1N4148, Corne73:D_SOD-123, B.Cu at (175.6, 49.2)
- added D39: 1N4148, Corne73:D_SOD-123, B.Cu at (283.2, 80.2)
- added D40: 1N4148, Corne73:D_SOD-123, B.Cu at (264.2, 80.2)
- added D41: 1N4148, Corne73:D_SOD-123, B.Cu at (245.1, 75.4)
- added D42: 1N4148, Corne73:D_SOD-123, B.Cu at (235.5, 63.6)
- added D43: 1N4148, Corne73:D_SOD-123, B.Cu at (207.0, 75.4)
- added D44: 1N4148, Corne73:D_SOD-123, B.Cu at (188.0, 77.8)
- added D45: 1N4148, Corne73:D_SOD-123, B.Cu at (225.3, 100.0)
- added D46: 1N4148, Corne73:D_SOD-123, B.Cu at (196.0, 100.9)
- added D47: 1N4148, Corne73:D_SOD-123, B.Cu at (181.6, 105.8)
- added D48: 1N4148, Corne73:D_SOD-123, B.Cu at (175.6, 68.2)
- added F2: Fuse_Small, Fuse:Fuse_1206_3216Metric, B.Cu at (181.2, 36.9)
- added J4: nice!view, Connector_PinHeader_2.54mm:PinHeader_1x05_P2.54mm_Vertical, B.Cu at (177.4, 76.3)
- added J5: Battery, Connector_Molex:Molex_Pico-EZmate_78171-0002_1x02-1MP_P1.20mm_Vertical, B.Cu at (181.7, 74.1)
- added J6: TC2030_SWD, PCM_marbastlib-various:CON_TC2030_outlined, B.Cu at (240.2, 79.5)
- added L2: 10 uH, Inductor_SMD:L_0603_1608Metric, B.Cu at (225.8, 73.3)
- added LED2: CHARGE, LED_SMD:LED_0805_2012Metric, B.Cu at (163.3, 88.3)
- added Q2: AO3401A, Package_TO_SOT_SMD:SOT-23, B.Cu at (169.0, 82.6)
- added R4: 10k, Resistor_SMD:R_0603_1608Metric, B.Cu at (181.7, 84.5)
- added R5: 5k, Resistor_SMD:R_0603_1608Metric, B.Cu at (172.2, 84.6)
- added R6: 5k, Resistor_SMD:R_0603_1608Metric, B.Cu at (171.5, 87.6)
- added SW24: SW_Push, PCM_marbastlib-various:SW_T1A2QR, B.Cu at (231.5, 74.6)
- added SW25: SW_SPDT, Button_Switch_SMD:SW_SPDT_PCM12, B.Cu at (164.3, 82.1)
- added U1: USBLC6-2SC6, Package_TO_SOT_SMD:SOT-23-6, B.Cu at (182.8, 42.7)
- added U4: TP4056, qw-footprints:CustomTP4056, B.Cu at (177.0, 84.8)
- added U5: nRF52840_E73-2G4M08S1C, PCM_marbastlib-various:nRF52840_E73-2G4M08S1C, B.Cu at (229.7, 85.1)
- added Y2: 32.768 KHz, Crystal:Crystal_SMD_2012-2Pin_2.0x1.2mm, B.Cu at (219.6, 80.6)
- BT1, BT2, BT3, BT4, rBT1, rBT2, rBT3, rBT4: footprint kbd_local:Breakaway_Tabs -> Corne73:Breakaway_Tabs
- H1, H2, H5, H6: moved to B.Cu
- SW23: footprint Button_Switch_SMD:SW_SPST_SKQG_WithStem -> PCM_marbastlib-various:SW_T1A2QR
- rEXSW1, rEXSW2: footprint kbd_local:keyswitch_cherrymx_hotswap_1u_rotary_encoder_ec12 -> Corne73:SwitchCombo+Encoder; moved to F.Cu
- rSW1, rSW8, rSW9: moved to F.Cu
- moved H5 566.8 mm to (358.6, 53.8), turned to 180 degrees
- moved H1 564.7 mm to (357.6, 44.2), turned to 180 degrees
- moved H6 558.4 mm to (354.4, 53.8), turned to 180 degrees
- moved H2 552.9 mm to (351.7, 44.2), turned to 180 degrees
- moved H4 552.5 mm to (340.0, 44.2)
- moved H8 552.5 mm to (346.1, 53.8)
- moved H7 523.9 mm to (350.3, 53.8)
- moved H3 355.5 mm to (345.8, 44.2)
- moved rBT4 165.0 mm to (267.5, 88.6)
- moved BT1 165.0 mm to (67.5, 25.3)
- moved BT2 165.0 mm to (105.6, 25.3)
- moved BT3 165.0 mm to (29.4, 88.6)
- moved BT4 165.0 mm to (48.4, 88.6)
- moved C1 165.0 mm to (130.3, 79.0)
- moved C2 165.0 mm to (128.7, 79.0)
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- renumbered C7 to C1, C6 to C2, C8 to C3, C1 to C5, C2 to C6, C3 to C7, C5 to C8, J5 to J2, J6 to J3, J2 to J7, R6 to R3, R5 to R7, R7 to R8, U1 to U3, U3 to U6
Connections:
- net /right/D+ renamed DBUS+R
- net /right/D- renamed DBUS-R
- net /right/RE0A renamed /right/RE0BR
- J3 pad 1: GND -> +BATT
- J3 pad 2: +BATT -> GND
- U3 pad 14: unconnected-(U1-P0.06-Pad14) -> COL4
- U3 pad 35: COL4 -> COL5
- U3 pad 41: COL5 -> unconnected-(U3-P0.09/NFC1-Pad41)
- rEXSW1 pad B: /right/REB -> CSR
- rEXSW1 pad S1: GNDR -> COL6R
- rEXSW1 pad S2: /right/KEYEX1 -> Net-(D38-A)
- rEXSW2 pad A: /right/RE1A -> MOSIR
- rEXSW2 pad B: /right/REB -> SCKR
- rEXSW2 pad S1: GNDR -> COL6R
- rEXSW2 pad S2: /right/KEYEX2 -> Net-(D48-A)
- rSW1 pad 1: /right/KEY1 -> COL5R
- rSW1 pad 2: GNDR -> Net-(D47-A)
- rSW10 pad 1: /right/KEY10 -> Net-(D42-A)
- rSW10 pad 2: GNDR -> COL3R
- rSW11 pad 1: /right/KEY11 -> Net-(D35-A)
- rSW11 pad 2: GNDR -> COL3R
- rSW12 pad 1: /right/KEY12 -> Net-(D29-A)
- rSW12 pad 2: GNDR -> COL3R
- rSW13 pad 1: /right/KEY13 -> Net-(D28-A)
- rSW13 pad 2: GNDR -> COL2R
- rSW14 pad 1: /right/KEY14 -> Net-(D34-A)
- rSW14 pad 2: GNDR -> COL2R
- rSW15 pad 1: /right/KEY15 -> Net-(D41-A)
- rSW15 pad 2: GNDR -> COL2R
- rSW16 pad 1: /right/KEY16 -> Net-(D40-A)
- rSW16 pad 2: GNDR -> COL1R
- rSW17 pad 1: /right/KEY17 -> Net-(D33-A)
- rSW17 pad 2: GNDR -> COL1R
- rSW18 pad 1: /right/KEY18 -> Net-(D27-A)
- rSW18 pad 2: GNDR -> COL1R
- rSW19 pad 1: /right/KEY19 -> Net-(D26-A)
- rSW19 pad 2: GNDR -> COL0R
- rSW2 pad 1: /right/KEY2 -> Net-(D44-A)
- rSW2 pad 2: GNDR -> COL5R
- rSW20 pad 1: /right/KEY20 -> Net-(D32-A)
- rSW20 pad 2: GNDR -> COL0R
- rSW21 pad 1: /right/KEY21 -> Net-(D39-A)
- rSW21 pad 2: GNDR -> COL0R
- rSW3 pad 1: /right/KEY3 -> Net-(D37-A)
- rSW3 pad 2: GNDR -> COL5R
- rSW4 pad 1: /right/KEY4 -> Net-(D31-A)
- rSW4 pad 2: GNDR -> COL5R
- rSW5 pad 1: /right/KEY5 -> Net-(D30-A)
- rSW5 pad 2: GNDR -> COL4R
- rSW6 pad 1: /right/KEY6 -> Net-(D36-A)
- rSW6 pad 2: GNDR -> COL4R
- rSW7 pad 1: /right/KEY7 -> Net-(D43-A)
- rSW7 pad 2: GNDR -> COL4R
- rSW8 pad 1: /right/KEY8 -> Net-(D46-A)
- rSW8 pad 2: GNDR -> COL4R
- rSW9 pad 1: /right/KEY9 -> Net-(D45-A)
- rSW9 pad 2: GNDR -> COL3R
Routing:
- net +5VR: track 0.00 -> 170.6 mm, vias 0 -> 3
- net COL0R: track 0.00 -> 113.4 mm
- net ROW1R: track 0.00 -> 102.7 mm
- net ROW0R: track 0.00 -> 102.6 mm
- net COL5R: track 0.00 -> 99.0 mm
- net D-R: track 0.00 -> 96.0 mm
- net D+R: track 0.00 -> 95.8 mm
- net COL1R: track 0.00 -> 94.6 mm
- net +VSWR: track 0.00 -> 80.4 mm, vias 0 -> 2
- net COL4R: track 0.00 -> 77.2 mm
- net COL3R: track 0.00 -> 76.4 mm
- net ROW2R: track 0.00 -> 75.8 mm
- net COL2R: track 0.00 -> 72.8 mm
- net ROW3R: track 0.00 -> 56.4 mm
- net COL6R: track 0.00 -> 48.4 mm
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- added copper zone on B.Cu, net GNDR
- added copper zone on F.Cu, net GNDR
Other:
- outline, holes or cut-outs redrawn
- board text added: "When I started my journey into mechanical keyboads, the Corne was one of the first boards that popped into my feed. But I never had a Corne before. I made several attempts before but his is the only one that actually got built."
- board text removed: "Edge of body"
- board text removed: "ON OFF"
