File: PCB/cherry-hotswap/corne73.kicad_sch (KiCad schematic)
At the start: 0 parts

Commit message: Started work on right side
Parts:
- added H1, H2, H3, H4: qw-logo, qw-logo:qw new logo silk + copper sm, symbol Mechanical:MountingHole
- added H5, H6, H7, H8: 1999-logo, 1999:1999 logo md, symbol Mechanical:MountingHole
