File: PCB/common/left.kicad_sch (KiCad schematic)
At the start: 68 parts, among them J2 TRS, J3 TC2030_SWD, J4 Battery, Q1 AO3401A, SW22 SW_SPDT, SW23 SW_Push, U2 nRF52840_E73-2G4M08S1C, U3 TP4056, U3 USBLC6-2SC6, Y1 32.768 KHz

Commit message: Catching up
Parts:
- removed D2: LED_Dual_AKKA, symbol Device:LED_Dual_AKKA
- removed J2: TRS, kbd_local:PJ-398A-5A_PJ-399B-6A, symbol Connector_Audio:AudioJack3
- removed J?: Conn_01x04, kbd_local:OLED, symbol Connector_Generic:Conn_01x04
- removed J?: Conn_01x03, Connector_PinHeader_2.54mm:PinHeader_1x03_P2.54mm_Vertical, symbol Connector_Generic:Conn_01x03
- removed R4: 806, Resistor_SMD:R_0603_1608Metric, symbol Device:R_Small
- removed R5: 2M, Resistor_SMD:R_0603_1608Metric, symbol Device:R_Small
- removed ZD?: RB521S30T1G, Diode_SMD:D_SOD-523, symbol Diode:ESD5Zxx
- added D10, D11, D12, D13, D14, D15, D16, D17, D18, D19, D2, D20, D21, D22, D23, D24, D3, D4, D5, D6, D7, D8, D9: 1N4148, qw-footprints:CUSTOM D_SOD-123, symbol Device:D_Small
- added F1: Fuse_Small, Fuse:Fuse_1206_3216Metric, symbol Device:Fuse_Small
- added J2: nice!view, Connector_PinHeader_2.54mm:PinHeader_1x05_P2.54mm_Vertical, symbol Connector_Generic:Conn_01x05
- SW1: renamed from SW?; footprint kbd:keyswitch_cherrymx_hotswap_1.5u -> PCM_marbastlib-mx:SW_MX_HS_CPG151101S11_1.5u
- SW10, SW11, SW12, SW13, SW14, SW15, SW16, SW17, SW18, SW19, SW2, SW20, SW21, SW3, SW4, SW5, SW6, SW7, SW8, SW9: renamed from SW?; footprint kbd:keyswitch_cherrymx_hotswap_1u -> PCM_marbastlib-mx:SW_MX_HS_CPG151101S11_1u
- gave numbers to parts that had none: 5
- renumbered C12 to C1, C13 to C2, C10 to C3, C9 to C4, C11 to C5, C1 to C6, C2 to C7, C6 to C8, D24 to D1, H10 to H1, H11 to H2, H12 to H3, H13 to H4, H14 to H5, H15 to H6, H16 to H7, H17 to H8, J3 to J5, J4 to J6, L2 to L1, R2 to R5, R1 to R6, R3 to R7, U2 to U1, U3 to U2
Connections:
- net BATTTON is gone; now on an unnamed net: Q1.3 (D)
- net +5V: now also F1.2
- net +BATT: now also SW22.1 (A)
- net D+: now also U3.1 (I/O1); no longer U3.4 (I/O2)
- net DBUS-: now also U3.4 (I/O2); no longer U3.1 (I/O1)
- net GND: now also SW23.2, J2.2 (Pin_2); no longer EXSW1.S1, EXSW2.S1, SW1.2, SW10.2, SW11.2, SW12.2, SW13.2, SW14.2, SW15.2, SW16.2, SW17.2, SW18.2, SW19.2, SW2.2, SW20.2, SW21.2, SW3.2, SW4.2, SW5.2, SW6.2, SW7.2, SW8.2, SW9.2
- net RESET: now also SW23.1
- net VBUS: now also F1.1
- net VDD: now also J2.3 (Pin_3)
- net 0.02: no longer names the net of U1.7 (P0.02/AIN0)
- net 0.03: no longer names the net of U1.3 (P0.03/AIN1)
- net 0.04: no longer names the net of U1.18 (P0.04/AIN2)
- net 0.06 renamed CS
- net CS: now also J2.1 (Pin_1)
- net 0.07: no longer names the net of U1.22 (P0.07)
- net 0.08: no longer names the net of U1.16 (P0.08)
- net 0.09: no longer names the net of U1.41 (P0.09/NFC1)
- net 0.10: no longer names the net of U1.43 (P0.10/NFC2)
- net 0.12: no longer names the net of U1.20 (P0.12)
- net 0.13: no longer names the net of U1.33 (P0.13)
- net 0.15: no longer names the net of U1.28 (P0.15)
- net 0.17 renamed MOSI
- net MOSI: now also J2.5 (Pin_5)
- net 0.20 renamed SCK
- net SCK: now also J2.4 (Pin_4)
- net 0.22: no longer names the net of U1.34 (P0.22)
- net 0.24: no longer names the net of U1.35 (P0.24)
- net 0.26: no longer names the net of U1.12 (P0.26)
- net 0.28: no longer names the net of U1.4 (P0.28/AIN4)
- net 0.29: no longer names the net of U1.8 (P0.29/AIN5)
- net 0.30: no longer names the net of U1.10 (P0.30/AIN6)
- net 0.31: no longer names the net of U1.9 (P0.31/AIN7)
- net 1.00: no longer names the net of U1.36 (P1.00)
- net 1.02: no longer names the net of U1.38 (P1.02)
- net 1.04: no longer names the net of U1.40 (P1.04)
- net 1.06: no longer names the net of U1.42 (P1.06)
- net 1.09: no longer names the net of U1.17 (P1.09)
- net 1.10: no longer names the net of U1.2 (P1.10)
- net 1.11: no longer names the net of U1.1 (P1.11)
- net 1.13: no longer names the net of U1.6 (P1.13)
- net KEY1: no longer names the net of SW1.1
- net KEY1: now also D22.2 (A)
- net KEY10: no longer names the net of SW10.1
- net KEY10: now also D17.2 (A)
- net KEY11: no longer names the net of SW11.1
- net KEY11: now also D11.2 (A)
- net KEY12: no longer names the net of SW12.1
- net KEY12: now also D5.2 (A)
- net KEY13: no longer names the net of SW13.1
- net KEY13: now also D4.2 (A)
- net KEY14: no longer names the net of SW14.1
- net KEY14: now also D10.2 (A)
- net KEY15: no longer names the net of SW15.1
- net KEY15: now also D16.2 (A)
- net KEY16: no longer names the net of SW16.1
- net KEY16: now also D15.2 (A)
- net KEY17: no longer names the net of SW17.1
- net KEY17: now also D9.2 (A)
- net KEY18: no longer names the net of SW18.1
- net KEY18: now also D3.2 (A)
- net KEY19: no longer names the net of SW19.1
- net KEY19: now also D2.2 (A)
- net KEY2: no longer names the net of SW2.1
- net KEY2: now also D19.2 (A)
- net KEY20: no longer names the net of SW20.1
- net KEY20: now also D8.2 (A)
- net KEY21: no longer names the net of SW21.1
- net KEY21: now also D14.2 (A)
- net KEY3: no longer names the net of SW3.1
- net KEY3: now also D13.2 (A)
- net KEY4: no longer names the net of SW4.1
- net KEY4: now also D7.2 (A)
- net KEY5: no longer names the net of SW5.1
- net KEY5: now also D6.2 (A)
- net KEY6: no longer names the net of SW6.1
- net KEY6: now also D12.2 (A)
- net KEY7: no longer names the net of SW7.1
- net KEY7: now also D18.2 (A)
- net KEY8: no longer names the net of SW8.1
- net KEY8: now also D21.2 (A)
- net KEY9: no longer names the net of SW9.1
- net KEY9: now also D20.2 (A)
- net KEYEX1: no longer names the net of EXSW1.S2
- net KEYEX2: no longer names the net of EXSW2.S2
- net VSENSE: no longer names the net of U1.15 (P0.05/AIN3)
- new net: D2.1 (K), D3.1 (K), D4.1 (K), D5.1 (K), D6.1 (K), D7.1 (K)
- new net: SW5.2, SW6.2, SW7.2, SW8.2
- new net: D20.1 (K), D21.1 (K), D22.1 (K), D24.1 (K)
- new net: SW1.2, SW2.2, SW3.2, SW4.2
- new net: D10.1 (K), D11.1 (K), D12.1 (K), D13.1 (K), D23.1 (K), D8.1 (K), D9.1 (K)
- new net: SW10.2, SW11.2, SW12.2, SW9.2
- new net: SW19.2, SW20.2, SW21.2
- new net: D14.1 (K), D15.1 (K), D16.1 (K), D17.1 (K), D18.1 (K), D19.1 (K)
- new net: SW13.2, SW14.2, SW15.2
- new net: SW16.2, SW17.2, SW18.2
- new net: D24.2 (A), EXSW2.S1
- new net: D23.2 (A), EXSW1.S1
Other:
- note removed: "DEBUG"
- note removed: "OLED"
- note removed: "TRS"
- note removed: "VBUS ESD"
- moved on the sheet: D1, EXSW1, Q1, R6, SW1, SW10, SW11, SW12, SW13, SW14, SW15, SW16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

Commit message: Changed footprints, made decisions
Parts:
- D1: footprint Diode_SMD:D_SOD-323 -> Corne73:D_SOD-123
- D10, D11, D12, D13, D14, D15, D16, D17, D18, D19, D2, D20, D21, D22, D23, D24, D3, D4, D5, D6, D7, D8, D9: footprint qw-footprints:CUSTOM D_SOD-123 -> Corne73:D_SOD-123
- SW1: footprint PCM_marbastlib-mx:SW_MX_HS_CPG151101S11_1.5u -> Corne73:SwitchCombo
- SW10, SW11, SW12, SW13, SW14, SW15, SW16, SW17, SW18, SW19, SW2, SW20, SW21, SW3, SW4, SW5, SW6, SW7, SW8, SW9: footprint PCM_marbastlib-mx:SW_MX_HS_CPG151101S11_1u -> Corne73:SwitchCombo
Changed lines of the file:
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@@
 		)
 		(instances
-			(project ""
+			(project "corne73"
 				(path "/4cc5d416-57f5-4147-8183-e03ae6b1198a/089db7cd-2934-428b-a62a-55e0735649ba"
 					(reference "J2")
@@
 			)
 		)
-		(property "Footprint" "qw-footprints:CUSTOM D_SOD-123"
+		(property "Footprint" "Corne73:D_SOD-123"
 			(at 373.38 182.88 90)
 			(effects
@@
 			)
 		)
-		(property "Footprint" "PCM_marbastlib-mx:SW_MX_HS_CPG151101S11_1u"
+		(property "Footprint" "Corne73:SwitchCombo"
 			(at 354.33 175.26 0)
 			(effects
@@
 			)
 		)
-		(property "Footprint" "qw-footprints:CUSTOM D_SOD-123"
+		(property "Footprint" "Corne73:D_SOD-123"
 			(at 373.38 226.06 90)
 			(effects
@@
 			)
 		)
-		(property "Footprint" "PCM_marbastlib-mx:SW_MX_HS_CPG151101S11_1u"
+		(property "Footprint" "Corne73:SwitchCombo"
 			(at 368.3 175.26 0)
 			(effects
@@
 			)
 		)
-		(property "Footprint" "qw-footprints:CUSTOM D_SOD-123"
+		(property "Footprint" "Corne73:D_SOD-123"
 			(at 359.41 196.85 90)
 			(effects
@@
 			)
 		)
-		(property "Footprint" "PCM_marbastlib-mx:SW_MX_HS_CPG151101S11_1u"
+		(property "Footprint" "Corne73:SwitchCombo"
 			(at 340.36 175.26 0)
 			(effects
@@
 			)
 		)
-		(property "Footprint" "PCM_marbastlib-mx:SW_MX_HS_CPG151101S11_1u"
+		(property "Footprint" "Corne73:SwitchCombo"
 			(at 354.33 204.47 0)
 			(effects
@@
 			)
 		)
-		(property "Footprint" "qw-footprints:CUSTOM D_SOD-123"
+		(property "Footprint" "Corne73:D_SOD-123"
 			(at 300.99 182.88 90)
 			(effects
@@
 		)
 		(instances
-			(project ""
+			(project "corne73"
 				(path "/4cc5d416-57f5-4147-8183-e03ae6b1198a/089db7cd-2934-428b-a62a-55e0735649ba"
 					(reference "D2")
@@
 			)
 		)
-		(property "Footprint" "qw-footprints:CUSTOM D_SOD-123"
+		(property "Footprint" "Corne73:D_SOD-123"
 			(at 373.38 196.85 90)
 			(effects
@@
 			)
 		)
-		(property "Footprint" "PCM_marbastlib-mx:SW_MX_HS_CPG151101S11_1u"
+		(property "Footprint" "Corne73:SwitchCombo"
 			(at 295.91 204.47 0)
 			(effects
@@
 			)
 		)
-		(property "Footprint" "qw-footprints:CUSTOM D_SOD-123"
+		(property "Footprint" "Corne73:D_SOD-123"
 			(at 300.99 212.09 90)
 			(effects
@@
 			)
 		)
-		(property "Footprint" "PCM_marbastlib-mx:SW_MX_HS_CPG151101S11_1u"
+		(property "Footprint" "Corne73:SwitchCombo"
 			(at 295.91 175.26 0)
 			(effects
@@
 			)
 		)
-		(property "Footprint" "qw-footprints:CUSTOM D_SOD-123"
+		(property "Footprint" "Corne73:D_SOD-123"
 			(at 345.44 196.85 90)
 			(effects
@@
 			)
 		)
-		(property "Footprint" "PCM_marbastlib-mx:SW_MX_HS_CPG151101S11_1u"
+		(property "Footprint" "Corne73:SwitchCombo"
 			(at 354.33 189.23 0)
 			(effects
@@
 			)
 		)
-		(property "Footprint" "PCM_marbastlib-mx:SW_MX_HS_CPG151101S11_1.5u"
+		(property "Footprint" "Corne73:SwitchCombo"
 			(at 368.3 218.44 0)
 			(effects
@@
 			)
 		)
-		(property "Footprint" "PCM_marbastlib-mx:SW_MX_HS_CPG151101S11_1u"
+		(property "Footprint" "Corne73:SwitchCombo"
 			(at 325.12 189.23 0)
 			(effects
@@
 			)
 		)
-		(property "Footprint" "PCM_marbastlib-mx:SW_MX_HS_CPG151101S11_1u"
+		(property "Footprint" "Corne73:SwitchCombo"
 			(at 309.88 189.23 0)
 			(effects
@@
 			)
 		)
-		(property "Footprint" "qw-footprints:CUSTOM D_SOD-123"
+		(property "Footprint" "Corne73:D_SOD-123"
 			(at 314.96 182.88 90)
 			(effects
@@
 			)
 		)
-		(property "Footprint" "qw-footprints:CUSTOM D_SOD-123"
+		(property "Footprint" "Corne73:D_SOD-123"
 			(at 345.44 212.09 90)
 			(effects
@@
 			)
 		)
-		(property "Footprint" "qw-footprints:CUSTOM D_SOD-123"
+		(property "Footprint" "Corne73:D_SOD-123"
 			(at 359.41 226.06 90)
 			(effects
@@
 			)
 		)
-		(property "Footprint" "qw-footprints:CUSTOM D_SOD-123"
+		(property "Footprint" "Corne73:D_SOD-123"
 			(at 330.2 182.88 90)
 			(effects
@@
 			)
 		)
-		(property "Footprint" "PCM_marbastlib-mx:SW_MX_HS_CPG151101S11_1u"
+		(property "Footprint" "Corne73:SwitchCombo"
 			(at 309.88 204.47 0)
 			(effects
@@
 			)
 		)
-		(property "Footprint" "PCM_marbastlib-mx:SW_MX_HS_CPG151101S11_1u"
+		(property "Footprint" "Corne73:SwitchCombo"
 			(at 325.12 204.47 0)
 			(effects
@@
 			)
 		)
-		(property "Footprint" "PCM_marbastlib-mx:SW_MX_HS_CPG151101S11_1u"
+		(property "Footprint" "Corne73:SwitchCombo"
 			(at 309.88 175.26 0)
 			(effects
@@
 			)
 		)
-		(property "Footprint" "qw-footprints:CUSTOM D_SOD-123"
+		(property "Footprint" "Corne73:D_SOD-123"
 			(at 300.99 196.85 90)
 			(effects
@@
 			)
 		)
-		(property "Footprint" "qw-footprints:CUSTOM D_SOD-123"
+		(property "Footprint" "Corne73:D_SOD-123"
 			(at 330.2 212.09 90)
 			(effects
@@
 			)
 		)
-		(property "Footprint" "qw-footprints:CUSTOM D_SOD-123"
+		(property "Footprint" "Corne73:D_SOD-123"
 			(at 345.44 226.06 90)
 			(effects
@@
 			)
 		)
-		(property "Footprint" "PCM_marbastlib-mx:SW_MX_HS_CPG151101S11_1u"
+		(property "Footprint" "Corne73:SwitchCombo"
 			(at 368.3 204.47 0)
 			(effects
@@
 			)
 		)
-		(property "Footprint" "qw-footprints:CUSTOM D_SOD-123"
+		(property "Footprint" "Corne73:D_SOD-123"
 			(at 359.41 212.09 90)
 			(effects
@@
 			)
 		)
-		(property "Footprint" "qw-footprints:CUSTOM D_SOD-123"
+		(property "Footprint" "Corne73:D_SOD-123"
 			(at 330.2 196.85 90)
 			(effects
@@
 			)
 		)
-		(property "Footprint" "qw-footprints:CUSTOM D_SOD-123"
+		(property "Footprint" "Corne73:D_SOD-123"
 			(at 345.44 182.88 90)
 			(effects
@@
 			)
 		)
-		(property "Footprint" "qw-footprints:CUSTOM D_SOD-123"
+		(property "Footprint" "Corne73:D_SOD-123"
 			(at 314.96 196.85 90)
 			(effects
@@
 			)
 		)
-		(property "Footprint" "qw-footprints:CUSTOM D_SOD-123"
+		(property "Footprint" "Corne73:D_SOD-123"
 			(at 391.16 238.76 90)
 			(effects
@@
 			)
 		)
-		(property "Footprint" "qw-footprints:CUSTOM D_SOD-123"
+		(property "Footprint" "Corne73:D_SOD-123"
 			(at 373.38 212.09 90)
 			(effects
@@
 			)
 		)
-		(property "Footprint" "PCM_marbastlib-mx:SW_MX_HS_CPG151101S11_1u"
+		(property "Footprint" "Corne73:SwitchCombo"
 			(at 340.36 189.23 0)
 			(effects
@@
 			)
 		)
-		(property "Footprint" "PCM_marbastlib-mx:SW_MX_HS_CPG151101S11_1u"
+		(property "Footprint" "Corne73:SwitchCombo"
 			(at 295.91 189.23 0)
 			(effects
@@
 			)
 		)
-		(property "Footprint" "Diode_SMD:D_SOD-323"
+		(property "Footprint" "Corne73:D_SOD-123"
 			(at 116.586 237.236 90)
 			(effects
@@
 			)
 		)
-		(property "Footprint" "qw-footprints:CUSTOM D_SOD-123"
+		(property "Footprint" "Corne73:D_SOD-123"
 			(at 359.41 182.88 90)
 			(effects
@@
 			)
 		)
-		(property "Footprint" "PCM_marbastlib-mx:SW_MX_HS_CPG151101S11_1u"
+		(property "Footprint" "Corne73:SwitchCombo"
 			(at 325.12 175.26 0)
 			(effects
@@
 			)
 		)
-		(property "Footprint" "PCM_marbastlib-mx:SW_MX_HS_CPG151101S11_1u"
+		(property "Footprint" "Corne73:SwitchCombo"
 			(at 354.33 218.44 0)
 			(effects
@@
 			)
 		)
-		(property "Footprint" "qw-footprints:CUSTOM D_SOD-123"
+		(property "Footprint" "Corne73:D_SOD-123"
 			(at 391.16 199.39 90)
 			(effects
@@
 			)
 		)
-		(property "Footprint" "PCM_marbastlib-mx:SW_MX_HS_CPG151101S11_1u"
+		(property "Footprint" "Corne73:SwitchCombo"
 			(at 340.36 218.44 0)
 			(effects
@@
 			)
 		)
-		(property "Footprint" "qw-footprints:CUSTOM D_SOD-123"
+		(property "Footprint" "Corne73:D_SOD-123"
 			(at 314.96 212.09 90)
 			(effects
@@
 		)
 		(instances
-			(project ""
+			(project "corne73"
 				(path "/4cc5d416-57f5-4147-8183-e03ae6b1198a/089db7cd-2934-428b-a62a-55e0735649ba"
 					(reference "#PWR020")
@@
 			)
 		)
-		(property "Footprint" "PCM_marbastlib-mx:SW_MX_HS_CPG151101S11_1u"
+		(property "Footprint" "Corne73:SwitchCombo"
 			(at 368.3 189.23 0)
 			(effects
@@
 			)
 		)
-		(property "Footprint" "PCM_marbastlib-mx:SW_MX_HS_CPG151101S11_1u"
+		(property "Footprint" "Corne73:SwitchCombo"
 			(at 340.36 204.47 0)
 			(effects

Commit message: More changes
Parts:
- EXSW1, EXSW2: footprint kbd_local:keyswitch_cherrymx_hotswap_1u_rotary_encoder_ec12 -> Corne73:SwitchCombo+Encoder
Connections:
- net RE0A is gone; now on net CS: EXSW1.A
- net RE1A is gone; now on net SCK: EXSW2.A
- net MOSI: now also EXSW2.B
- net RESET: no longer J5.3 (~{RST})
- net at D20.1 (K), D21.1 (K), D22.1 (K): no longer D24.1 (K)
- net at D14.1 (K), D15.1 (K), D16.1 (K)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: now also D24.1 (K)
- net at EXSW2.S2: now also EXSW1.S2
- net REB renamed RE0B
- net RE0B: no longer EXSW2.B
- no-connect marks 4 -> 5
Other:
- note added: "Display"
- note added: "USB C"
- note removed: "Extention"
- note removed: "POWER"
- moved on the sheet: J2, J5

Commit message: Left hand routed
Connections:
- net CS: now also U1.12 (P0.26); no longer U1.14 (P0.06)
- net MOSI: now also U1.17 (P1.09); no longer U1.30 (P0.17)
- net RE0B: now also U1.10 (P0.30/AIN6)
- net SCK: now also U1.15 (P0.05/AIN3); no longer U1.32 (P0.20)
- net COL3: now reaches U1.1 (P1.11)
- net COL3: now also SW10.2, SW11.2, SW12.2, SW9.2
- net ROW2: now reaches U1.2 (P1.10)
- net ROW2: now also D14.1 (K), D15.1 (K), D16.1 (K), D17.1 (K), D18.1 (K), D19.1 (K), D24.1 (K)
- net COL2: now reaches U1.3 (P0.03/AIN1)
- net COL2: now also SW13.2, SW14.2, SW15.2
- net ROW3: now reaches U1.33 (P0.13)
- net ROW3: now also D20.1 (K), D21.1 (K), D22.1 (K)
- net COL4: now reaches U1.35 (P0.24)
- net COL4: now also SW5.2, SW6.2, SW7.2, SW8.2
- net COL1: now reaches U1.4 (P0.28/AIN4)
- net COL1: now also SW16.2, SW17.2, SW18.2
- net COL5: now reaches U1.41 (P0.09/NFC1)
- net COL5: now also SW1.2, SW2.2, SW3.2, SW4.2
- net COL0: now reaches U1.6 (P1.13)
- net COL0: now also SW19.2, SW20.2, SW21.2
- net ROW1: now reaches U1.7 (P0.02/AIN0)
- net ROW1: now also D10.1 (K), D11.1 (K), D12.1 (K), D13.1 (K), D23.1 (K), D8.1 (K), D9.1 (K)
- net ROW0: now reaches U1.8 (P0.29/AIN5)
- net ROW0: now also D2.1 (K), D3.1 (K), D4.1 (K), D5.1 (K), D6.1 (K), D7.1 (K)
- net COL6: now reaches U1.9 (P0.31/AIN7)
- net COL6: now also EXSW1.S2, EXSW2.S2
Other:
- moved on the sheet: C1, C2, C3, C4, C5, J5, L1, U1, Y1

Commit message: Started work on right side
Parts:
- removed H1, H2, H3, H4: qw-logo, qw-logo:qw new logo silk + copper sm, symbol Mechanical:MountingHole
- removed H5, H6, H7, H8: 1999-logo, 1999:1999 logo md, symbol Mechanical:MountingHole
- BT1, BT2, BT3, BT4: footprint kbd_local:Breakaway_Tabs -> Corne73:Breakaway_Tabs
- SW23: footprint Button_Switch_SMD:SW_SPST_SKQG_WithStem -> PCM_marbastlib-various:SW_T1A2QR
- renumbered C7 to C1, C6 to C2, C8 to C3, C1 to C5, C2 to C6, C3 to C7, C5 to C8, J5 to J2, J6 to J3, J2 to J7, R6 to R3, R5 to R7, R7 to R8, U1 to U3, U3 to U6
Connections:
- net +BATT: now also J3.1 (Pin_1); no longer J3.2 (Pin_2)
- net COL4: now also U3.14 (P0.06); no longer U3.35 (P0.24)
- net COL5: now also U3.35 (P0.24); no longer U3.41 (P0.09/NFC1)
- net GND: now also J3.2 (Pin_2); no longer J3.1 (Pin_1)
- no-connect marks 5 -> 6
Other:
- note added: "Battery Charging"
- note added: "E73-2G4M08S1C"
- note added: "ESD Protection"
- note added: "Power Path"
- note added: "Switch Matrix"
- note removed: "Key switches"
- moved on the sheet: BT1, BT2, BT3, BT4, C1, C2, C3, C4, C5, C6, C7, C8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
