File: PCB/common/right.kicad_sch (KiCad schematic)
At the start: 35 parts, among them J2 TRS

Commit message: Catching up
Parts:
- rSW1: renamed from rSW?; footprint kbd:keyswitch_cherrymx_hotswap_1.5u -> PCM_marbastlib-mx:SW_MX_HS_CPG151101S11_1.5u
- rSW10, rSW11, rSW12, rSW13, rSW14, rSW15, rSW16, rSW17, rSW18, rSW19, rSW2, rSW20, rSW21, rSW3, rSW4, rSW5, rSW6, rSW7, rSW8, rSW9: renamed from rSW?; footprint kbd:keyswitch_cherrymx_hotswap_1u -> PCM_marbastlib-mx:SW_MX_HS_CPG151101S11_1u
- gave numbers to parts that had none: 9
- renumbered J2 to rJ2

Commit message: Changed footprints, made decisions
Parts:
- rSW1: footprint PCM_marbastlib-mx:SW_MX_HS_CPG151101S11_1.5u -> Corne73:SwitchCombo
- rSW10, rSW11, rSW12, rSW13, rSW14, rSW15, rSW16, rSW17, rSW18, rSW19, rSW2, rSW20, rSW21, rSW3, rSW4, rSW5, rSW6, rSW7, rSW8, rSW9: footprint PCM_marbastlib-mx:SW_MX_HS_CPG151101S11_1u -> Corne73:SwitchCombo
Changed lines of the file:
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@@
 			)
 		)
-		(property "Footprint" "PCM_marbastlib-mx:SW_MX_HS_CPG151101S11_1u"
+		(property "Footprint" "Corne73:SwitchCombo"
 			(at 236.22 118.11 0)
 			(effects
@@
 			)
 		)
-		(property "Footprint" "PCM_marbastlib-mx:SW_MX_HS_CPG151101S11_1u"
+		(property "Footprint" "Corne73:SwitchCombo"
 			(at 248.92 102.87 0)
 			(effects
@@
 			)
 		)
-		(property "Footprint" "PCM_marbastlib-mx:SW_MX_HS_CPG151101S11_1u"
+		(property "Footprint" "Corne73:SwitchCombo"
 			(at 236.22 102.87 0)
 			(effects
@@
 			)
 		)
-		(property "Footprint" "PCM_marbastlib-mx:SW_MX_HS_CPG151101S11_1u"
+		(property "Footprint" "Corne73:SwitchCombo"
 			(at 198.12 133.35 0)
 			(effects
@@
 			)
 		)
-		(property "Footprint" "PCM_marbastlib-mx:SW_MX_HS_CPG151101S11_1u"
+		(property "Footprint" "Corne73:SwitchCombo"
 			(at 210.82 133.35 0)
 			(effects
@@
 			)
 		)
-		(property "Footprint" "PCM_marbastlib-mx:SW_MX_HS_CPG151101S11_1.5u"
+		(property "Footprint" "Corne73:SwitchCombo"
 			(at 248.92 148.59 0)
 			(effects
@@
 			)
 		)
-		(property "Footprint" "PCM_marbastlib-mx:SW_MX_HS_CPG151101S11_1u"
+		(property "Footprint" "Corne73:SwitchCombo"
 			(at 198.12 118.11 0)
 			(effects
@@
 			)
 		)
-		(property "Footprint" "PCM_marbastlib-mx:SW_MX_HS_CPG151101S11_1u"
+		(property "Footprint" "Corne73:SwitchCombo"
 			(at 185.42 133.35 0)
 			(effects
@@
 			)
 		)
-		(property "Footprint" "PCM_marbastlib-mx:SW_MX_HS_CPG151101S11_1u"
+		(property "Footprint" "Corne73:SwitchCombo"
 			(at 223.52 148.59 0)
 			(effects
@@
 			)
 		)
-		(property "Footprint" "PCM_marbastlib-mx:SW_MX_HS_CPG151101S11_1u"
+		(property "Footprint" "Corne73:SwitchCombo"
 			(at 185.42 102.87 0)
 			(effects
@@
 			)
 		)
-		(property "Footprint" "PCM_marbastlib-mx:SW_MX_HS_CPG151101S11_1u"
+		(property "Footprint" "Corne73:SwitchCombo"
 			(at 248.92 133.35 0)
 			(effects
@@
 			)
 		)
-		(property "Footprint" "PCM_marbastlib-mx:SW_MX_HS_CPG151101S11_1u"
+		(property "Footprint" "Corne73:SwitchCombo"
 			(at 210.82 102.87 0)
 			(effects
@@
 			)
 		)
-		(property "Footprint" "PCM_marbastlib-mx:SW_MX_HS_CPG151101S11_1u"
+		(property "Footprint" "Corne73:SwitchCombo"
 			(at 236.22 133.35 0)
 			(effects
@@
 			)
 		)
-		(property "Footprint" "PCM_marbastlib-mx:SW_MX_HS_CPG151101S11_1u"
+		(property "Footprint" "Corne73:SwitchCombo"
 			(at 210.82 118.11 0)
 			(effects
@@
 			)
 		)
-		(property "Footprint" "PCM_marbastlib-mx:SW_MX_HS_CPG151101S11_1u"
+		(property "Footprint" "Corne73:SwitchCombo"
 			(at 248.92 118.11 0)
 			(effects
@@
 			)
 		)
-		(property "Footprint" "PCM_marbastlib-mx:SW_MX_HS_CPG151101S11_1u"
+		(property "Footprint" "Corne73:SwitchCombo"
 			(at 185.42 118.11 0)
 			(effects
@@
 			)
 		)
-		(property "Footprint" "PCM_marbastlib-mx:SW_MX_HS_CPG151101S11_1u"
+		(property "Footprint" "Corne73:SwitchCombo"
 			(at 223.52 118.11 0)
 			(effects
@@
 			)
 		)
-		(property "Footprint" "PCM_marbastlib-mx:SW_MX_HS_CPG151101S11_1u"
+		(property "Footprint" "Corne73:SwitchCombo"
 			(at 198.12 102.87 0)
 			(effects
@@
 			)
 		)
-		(property "Footprint" "PCM_marbastlib-mx:SW_MX_HS_CPG151101S11_1u"
+		(property "Footprint" "Corne73:SwitchCombo"
 			(at 236.22 148.59 0)
 			(effects
@@
 			)
 		)
-		(property "Footprint" "PCM_marbastlib-mx:SW_MX_HS_CPG151101S11_1u"
+		(property "Footprint" "Corne73:SwitchCombo"
 			(at 223.52 133.35 0)
 			(effects
@@
 			)
 		)
-		(property "Footprint" "PCM_marbastlib-mx:SW_MX_HS_CPG151101S11_1u"
+		(property "Footprint" "Corne73:SwitchCombo"
 			(at 223.52 102.87 0)
 			(effects

Commit message: More changes
Parts:
- removed rU3: TPD4E05U06DQAR, Package_SON:USON-10_2.5x1.0mm_P0.5mm, symbol Power_Protection:TPD4EUSB30
Other:
- note removed: "USB ESD"

Commit message: Started work on right side
Parts:
- removed rJ2: TRS, kbd_local:PJ-398A-5A_PJ-399B-6A, symbol Connector_Audio:AudioJack3
- removed rJ3: Conn_01x04, kbd_local:OLED, symbol Connector_Generic:Conn_01x04
- removed rJ4: Conn_01x03, Connector_PinHeader_2.54mm:PinHeader_1x03_P2.54mm_Vertical, symbol Connector_Generic:Conn_01x03
- removed rZD1: RB521S30T1G, Diode_SMD:D_SOD-523, symbol Diode:ESD5Zxx
- added C10, C12: 10uF, Capacitor_Tantalum_SMD:CP_EIA-2012-12_Kemet-R, symbol Device:C_Polarized_Small
- added C11, C14, C15: 4.7u, Capacitor_SMD:C_0603_1608Metric, symbol Device:C_Small
- added C13, C16: 12p, Capacitor_SMD:C_0603_1608Metric, symbol Device:C_Small
- added C9: 1u, Capacitor_SMD:C_0603_1608Metric, symbol Device:C_Small
- added D25: Schottky, Corne73:D_SOD-123, symbol Device:D_Schottky_Small
- added D26, D27, D28, D29, D30, D31, D32, D33, D34, D35, D36, D37, D38, D39, D40, D41, D42, D43, D44, D45, D46, D47, D48: 1N4148, Corne73:D_SOD-123, symbol Device:D_Small
- added F2: Fuse_Small, Fuse:Fuse_1206_3216Metric, symbol Device:Fuse_Small
- added J4: nice!view, Connector_PinHeader_2.54mm:PinHeader_1x05_P2.54mm_Vertical, symbol Connector_Generic:Conn_01x05
- added J5: Battery, Connector_Molex:Molex_Pico-EZmate_78171-0002_1x02-1MP_P1.20mm_Vertical, symbol Connector_Generic_MountingPin:Conn_01x02_MountingPin
- added J6: TC2030_SWD, PCM_marbastlib-various:CON_TC2030_outlined, symbol PCM_marbastlib-various:TC2030_SWD
- added L2: 10 uH, Inductor_SMD:L_0603_1608Metric, symbol Device:L_Small
- added LED2: CHARGE, LED_SMD:LED_0805_2012Metric, symbol Device:LED_Small
- added Q2: AO3401A, Package_TO_SOT_SMD:SOT-23, symbol Transistor_FET:AO3401A
- added R4: 10k, Resistor_SMD:R_0603_1608Metric, symbol Device:R_Small
- added R5, R6: 5k, Resistor_SMD:R_0603_1608Metric, symbol Device:R_Small
- added SW24: SW_Push, PCM_marbastlib-various:SW_T1A2QR, symbol Switch:SW_Push
- added SW25: SW_SPDT, Button_Switch_SMD:SW_SPDT_PCM12, symbol Switch:SW_SPDT
- added U1: USBLC6-2SC6, Package_TO_SOT_SMD:SOT-23-6, symbol Power_Protection:USBLC6-2SC6
- added U4: TP4056, qw-footprints:CustomTP4056, symbol PCM_marbastlib-various:TP4056
- added U5: nRF52840_E73-2G4M08S1C, PCM_marbastlib-various:nRF52840_E73-2G4M08S1C, symbol PCM_marbastlib-various:nRF52840_E73-2G4M08S1C
- added Y2: 32.768 KHz, Crystal:Crystal_SMD_2012-2Pin_2.0x1.2mm, symbol Device:Crystal_Small
- rBT1, rBT2, rBT3, rBT4: footprint kbd_local:Breakaway_Tabs -> Corne73:Breakaway_Tabs
- rEXSW1, rEXSW2: footprint kbd_local:keyswitch_cherrymx_hotswap_1u_rotary_encoder_ec12 -> Corne73:SwitchCombo+Encoder
Connections:
- net +5VR: now also C10.1, C11.1, C14.1, D25.2 (A), F2.2, LED2.2 (A), Q2.1 (G), R6.1, U1.5 (VBUS), U4.4 (VCC), U4.8 (CE), U5.27 (VBUS)
- net GNDR: now also C10.2, C11.2, C12.2, C13.2, C14.2, C15.2, C16.2, C9.2, J4.2 (Pin_2), J5.2 (Pin_2), J5.MP (MountPin), J6.5 (GND), R5.2, R6.2, SW24.2, U1.2 (GND), U4.1 (TEMP), U4.3 (GND), U5.21 (GND), U5.24 (GND), U5.5 (GND); no longer rEXSW1.S1, rEXSW2.S1, rSW1.2, rSW10.2, rSW11.2, rSW12.2, rSW13.2, rSW14.2, rSW15.2, rSW16.2, rSW17.2, rSW18.2, rSW19.2, rSW2.2, rSW20.2, rSW21.2, rSW3.2, rSW4.2, rSW5.2, rSW6.2, rSW7.2, rSW8.2, rSW9.2
- net VBUSR: now also F2.1
- net D+ renamed DBUS+R
- net DBUS+R: now also U1.6 (I/O1)
- net D- renamed DBUS-R
- net DBUS-R: now also U1.4 (I/O2)
- net KEY1 renamed COL5R
- net COL5R: now also rSW2.2, rSW3.2, rSW4.2, U5.4 (P0.28/AIN4)
- net KEY10: no longer names the net of rSW10.1
- net KEY10: now also D42.2 (A)
- net KEY11: no longer names the net of rSW11.1
- net KEY11: now also D35.2 (A)
- net KEY12: no longer names the net of rSW12.1
- net KEY12: now also D29.2 (A)
- net KEY13: no longer names the net of rSW13.1
- net KEY13: now also D28.2 (A)
- net KEY14: no longer names the net of rSW14.1
- net KEY14: now also D34.2 (A)
- net KEY15: no longer names the net of rSW15.1
- net KEY15: now also D41.2 (A)
- net KEY16: no longer names the net of rSW16.1
- net KEY16: now also D40.2 (A)
- net KEY17: no longer names the net of rSW17.1
- net KEY17: now also D33.2 (A)
- net KEY18: no longer names the net of rSW18.1
- net KEY18: now also D27.2 (A)
- net KEY19: no longer names the net of rSW19.1
- net KEY19: now also D26.2 (A)
- net KEY2: no longer names the net of rSW2.1
- net KEY2: now also D44.2 (A)
- net KEY20: no longer names the net of rSW20.1
- net KEY20: now also D32.2 (A)
- net KEY21: no longer names the net of rSW21.1
- net KEY21: now also D39.2 (A)
- net KEY3: no longer names the net of rSW3.1
- net KEY3: now also D37.2 (A)
- net KEY4: no longer names the net of rSW4.1
- net KEY4: now also D31.2 (A)
- net KEY5: no longer names the net of rSW5.1
- net KEY5: now also D30.2 (A)
- net KEY6: no longer names the net of rSW6.1
- net KEY6: now also D36.2 (A)
- net KEY7: no longer names the net of rSW7.1
- net KEY7: now also D43.2 (A)
- net KEY8: no longer names the net of rSW8.1
- net KEY8: now also D46.2 (A)
- net KEY9: no longer names the net of rSW9.1
- net KEY9: now also D45.2 (A)
- net KEYEX1: no longer names the net of rEXSW1.S2
- net KEYEX1: now also D38.2 (A)
- net KEYEX2: no longer names the net of rEXSW2.S2
- net KEYEX2: now also D48.2 (A)
- net RE0A renamed RE0BR
- net RE1A renamed MOSIR
- net MOSIR: now also J4.5 (Pin_5), U5.17 (P1.09)
- net REB renamed CSR
- net CSR: now also J4.1 (Pin_1), U5.12 (P0.26); no longer rEXSW2.B
- new net: D47.2 (A), rSW1.2
- new net: R5.1, U4.2 (PROG)
- new net: LED2.1 (K), R4.1
- new net: R4.2, U4.7 (CHRG)
- new net: C16.1, U5.13 (P0.01/XL2), Y2.1
- new net: C13.1, U5.11 (P0.00/XL1), Y2.2
- new net: Q2.3 (D), SW25.2 (B)
- new net +BATTR: C12.1, J5.1 (Pin_1), SW25.3 (C), U4.5 (BAT)
- new net +VSWR: C15.1, D25.1 (K), Q2.2 (S), U5.23 (VDDH)
- new net COL0R: U5.43 (P0.10/NFC2), rSW19.2, rSW20.2, rSW21.2
- new net COL1R: U5.33 (P0.13), rSW16.2, rSW17.2, rSW18.2
- new net COL2R: U5.35 (P0.24), rSW13.2, rSW14.2, rSW15.2
- new net COL3R: U5.2 (P1.10), rSW10.2, rSW11.2, rSW12.2, rSW9.2
- new net COL4R: U5.3 (P0.03/AIN1), rSW5.2, rSW6.2, rSW7.2, rSW8.2
- new net COL6R: rEXSW1.S1, rEXSW2.S1
- new net D+R: U1.1 (I/O1), U5.31 (D+)
- new net D-R: U1.3 (I/O2), U5.29 (D-)
- new net DCCHR: L2.1, U5.25 (DCCH)
- new net RESETR: SW24.1, U5.26 (P0.18/~{RESET})
- new net ROW0R: D26.1 (K), D27.1 (K), D28.1 (K), D29.1 (K), D30.1 (K), D31.1 (K)
- new net ROW1R: D32.1 (K), D33.1 (K), D34.1 (K), D35.1 (K), D36.1 (K), D37.1 (K), D38.1 (K)
- new net ROW2R: D39.1 (K), D40.1 (K), D41.1 (K), D42.1 (K), D43.1 (K), D44.1 (K), D48.1 (K), U5.41 (P0.09/NFC1)
- new net ROW3R: D45.1 (K), D46.1 (K), D47.1 (K), U5.1 (P1.11)
- new net SCKR: J4.4 (Pin_4), U5.15 (P0.05/AIN3), rEXSW2.B
- new net SWDCLKR: J6.4 (SWCLK), U5.39 (SWDCLK)
- new net SWDIOR: J6.2 (SWDIO), U5.37 (SWDIO)
- new net VDDR: C9.1, J4.3 (Pin_3), J6.1 (VCC), L2.2, U5.19 (VDD)
- no-connect marks 2 -> 6
Other:
- note added: "Battery Charging"
- note added: "Display"
- note added: "E73-2G4M08S1C"
- note added: "ESD Protection"
- note added: "Power Path"
- note added: "Programming header"
- note removed: "DEBUG"
- note removed: "Extention"
- note removed: "Key switches"
- note removed: "OLED"
- note removed: "TRS"
- note removed: "VBUS ESD"
- moved on the sheet: rEXSW1, rEXSW2, rSW1, rSW10, rSW11, rSW12, rSW13, rSW14, rSW15, rSW16, rSW17, rSW18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
